File: 6in-6out/6in-6out.kicad_pcb (KiCad board)
At the start: 2 copper layers, 150 x 70 mm, 227 parts, among them J1 S0, J10 COIL_0, J11 COIL_0, J12 COIL_0, J13 COIL_0, J14 COIL_0, J15 COIL_0, J16 COIL_0, J18 COIL_0, J19 Conn_01x04_Pin, J2 S0, J21 Conn_01x04_Pin, J22 Screw_Terminal_01x02, J23 COIL_0, J24 COIL_0, J25 COIL_0, J26 COIL_0, J27 COIL_0, J28 COIL_0, J29 COIL_0, J3 S0, J30 S0, J31 S0, J32 S0, J33 S0, J34 S0, J35 S0, J36 S0, J37 S0, J38 USB_C_Receptacle_USB2.0_16P, J4 S0, J5 S0, J6 S0, J7 S0, J8 S0, J9 COIL_0, M1 AO4828, M2 AO4828, M3 AO4828, M4 AO4828, M5 AO4828, M6 AO4828, M7 AO4828, M8 AO4828, Q1 MMBT2222A, Q2 MMBT2222A, SW3 SW_Push, U1 LTV-847, U10 LTV-847, U11 LTV-847, U12 LTV-847, U13 PCF8575DBR, U14 PCF8575DBR, U2 LTV-847, U3 MP2451DJ-LF-P, U4 ESP32-WROOM-32U, U5 LTV-847, U6 LTV-847, U7 AMS1117-3.3, U8 CH340C, U9 LTV-847

Commit message: Test Commit.
Parts:
- removed J29: COIL_0, JST-254:JST 2
Changed lines of the file:
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@@
-		)
-	)
-	(footprint "JST-254:JST 2"
-		(layer "F.Cu")
-		(at 126.0014 60.092)
-		(property "Reference" "J29"
-			(at 1.3716 -3.4036 0)
-			(unlocked yes)
-			(layer "F.SilkS")
-			(effects
-				(font
-					(size 1 1)
-					(thickness 0.1)
-				)
-			)
-		)
-		(property "Value" "COIL_0"
-			(at 1.3208 3.5052 0)
-			(unlocked yes)
-			(layer "F.Fab")
-			(effects
-				(font
-					(size 1 1)
-					(thickness 0.15)
-				)
-			)
-		)
-		(property "Footprint" "JST-254:JST 2"
-			(at 0 0 0)
-			(layer "F.Fab")
-			(hide yes)
-			(effects
-				(font
-					(size 1.27 1.27)
-					(thickness 0.15)
-				)
-			)
-		)
-		(property "Datasheet" ""
-			(at 0 0 0)
-			(layer "F.Fab")
-			(hide yes)
-			(effects
-				(font
-					(size 1.27 1.27)
-					(thickness 0.15)
-				)
-			)
-		)
-		(property "Description" "Generic connector, single row, 01x02, script generated (kicad-library-utils/schlib/autogen/connector/)"
-			(at 0 0 0)
-			(layer "F.Fab")
-			(hide yes)
-			(effects
-				(font
-					(size 1.27 1.27)
-					(thickness 0.15)
-				)
-			)
-		)
-		(property ki_fp_filters "Connector*:*_1x??_*")
-		(sheetname "output")
-		(sheetfile "output.kicad_sch")
-		(attr through_hole)
-		(fp_rect
-			(start -2.54 -2.54)
-			(end 5.0038 3.429)
-			(stroke
-				(width 0.1)
-				(type default)
-			)
-			(fill none)
-			(layer "F.SilkS")
-		)
-		(fp_rect
-			(start 0 -2.54)
-			(end 2.54 -1.524)
-			(stroke
-				(width 0.1)
-				(type default)
-			)
-			(fill none)
-			(layer "F.SilkS")
-		)
-		(fp_text user "${REFERENCE}"
-			(at 1.5748 1.7272 0)
-			(unlocked yes)
-			(layer "F.Fab")
-			(effects
-				(font
-					(size 1 1)
-					(thickness 0.15)
-				)
-			)
-		)
-		(pad "1" thru_hole roundrect
-			(at 0 0)
-			(size 1.7 1.7)
-			(drill 1)
-			(layers "*.Cu" "*.Mask")
-			(remove_unused_layers no)
-			(roundrect_rratio 0.25)
-			(net 23 "+24V")
-			(pinfunction "Pin_1")
-			(pintype "passive")
-		)
-		(pad "2" thru_hole circle
-			(at 2.54 0)
-			(size 1.7 1.7)
-			(drill 1)
-			(layers "*.Cu" "*.Mask")
-			(remove_unused_layers no)
-			(net 56 "Net-(D42-A)")
-			(pinfunction "Pin_2")
-			(pintype "passive")
-		)
-		(model "C:/Users/84886/Documents/KiCad/7.0/3dmodels/Thru Vertical/JST - XH - Thru (V) - 2Pin - 2.54mm.stp"
-			(offset
-				(xyz 1.25 0 0)
-			)
-			(scale
-				(xyz 1 1 1)
-			)
-			(rotate
-				(xyz 0 0 180)
-			)
 		)
 	)
