File: 6in-6out/MCU.kicad_sch (KiCad schematic)
At the start: 38 parts, among them J19 Conn_01x04_Pin, J21 Conn_01x04_Pin, J38 USB_C_Receptacle_USB2.0_16P, Q1 MMBT2222A, Q2 MMBT2222A, SW2 SW_DIP_x03, SW3 SW_Push, U4 ESP32-WROOM-32U, U7 AMS1117-3.3, U8 CH340C

Commit message: no message
Parts:
- Q1, Q2: value MMBT2222A -> S8050
Other:
- moved on the sheet: C10, Q1, Q2, R41, R6, R7, R82, R83, SW3, U4
