File: 6in-6out/output.kicad_sch (KiCad schematic)
At the start: 92 parts, among them J10 COIL_0, J11 COIL_0, J12 COIL_0, J13 COIL_0, J14 COIL_0, J15 COIL_0, J16 COIL_0, J18 COIL_0, J23 COIL_0, J24 COIL_0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

Commit message: no message
Other:
- moved on the sheet: D10, D11, D12, D13, D14, D15, D16, D17, D18, D19, D20, D21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
